Commit message: Prius Model: Adjusted to be more like the ADAS model.

File: src/prius_description/urdf/prius.urdf (robot description, URDF)
Before this commit: robot prius, 28 links, 27 joints
Links:
- removed link back_camera_link
- removed link back_camera_link_optical
- removed link back_left_far_sonar_link
- removed link back_left_middle_sonar_link
- removed link back_right_far_sonar_link
- removed link back_right_middle_sonar_link
- removed link front_left_far_sonar_link
- removed link front_left_laser_link
- removed link front_left_middle_sonar_link
- removed link front_right_far_sonar_link
- removed link front_right_laser_link
- removed link front_right_middle_sonar_link
- removed link left_camera_link
- removed link left_camera_link_optical
- removed link right_camera_link
- removed link right_camera_link_optical
Joints:
- removed joint back_camera_joint
- removed joint back_camera_optical_joint
- removed joint back_left_far_sonar_joint
- removed joint back_left_middle_sonar_joint
- removed joint back_right_far_sonar_joint
- removed joint back_right_middle_sonar_joint
- removed joint front_left_far_sonar_joint
- removed joint front_left_laser_joint
- removed joint front_left_middle_sonar_joint
- removed joint front_right_far_sonar_joint
- removed joint front_right_laser_joint
- removed joint front_right_middle_sonar_joint
- removed joint left_camera_joint
- removed joint left_camera_optical_joint
- removed joint right_camera_joint
- removed joint right_camera_optical_joint
- joint center_laser_joint: origin xyz=0 0.4 1.8 rpy=0 0 -1.5707 -> xyz=0 -2.3 0.6 rpy=0 0 -1.5707
- joint front_camera_joint: origin xyz=0 -0.4 1.4 rpy=0 0.05 -1.5707 -> xyz=0 -1 1.4 rpy=0 0.05 -1.5707

Commit message: Prius Model: Use GPU for lidar simulation.

File: src/prius_description/urdf/prius.urdf (robot description, URDF)
Before this commit: robot prius, 12 links, 11 joints
Joints:
- joint center_laser_joint: origin xyz=0 -2.3 0.6 rpy=0 0 -1.5707 -> xyz=0 -2.2 0.6 rpy=0 0 -1.5707

Commit message: Prius Model: Adjust camera to be more like the ADAS model.

File: src/prius_description/urdf/prius.urdf (robot description, URDF)
Before this commit: robot prius, 12 links, 11 joints
Joints:
- joint front_camera_joint: origin xyz=0 -1 1.4 rpy=0 0.05 -1.5707 -> xyz=0 -0.5 1.8 rpy=0 0.12 -1.5707

Commit message: Prius Model: Adjusted lidar orientation to match ADAS model.

File: src/prius_description/urdf/prius.urdf (robot description, URDF)
Before this commit: robot prius, 12 links, 11 joints
Joints:
- joint center_laser_joint: origin xyz=0 -2.2 0.6 rpy=0 0 -1.5707 -> xyz=0 -2.2 0.6 rpy=0 0 1.5707

Commit message: Prius Model: Now lightweight with super sticky wheels.

File: src/prius_description/urdf/prius.urdf (robot description, URDF)
Before this commit: robot prius, 12 links, 11 joints
Links:
- link base_link: mass 1 -> 0.1
- link chassis: mass 1356.0 -> 135.60
- link fl_axle: mass 1 -> .1
- link fr_axle: mass 1 -> .1
- link front_left_wheel: mass 11 -> 1.1
- link front_right_wheel: mass 11 -> 1.1
- link rear_left_wheel: mass 11 -> 1.1
- link rear_right_wheel: mass 11 -> 1.1
- link steering_wheel: mass 1.0 -> 0.10
